File: PCB/Final_Project_PCB/Final_Project_PCB.kicad_sch (KiCad schematic)
At the start: 14 parts

Commit message: Schematic Finished
Parts:
- added 01-GND_Breakout1, 46-GND_Breakout1: Conn_01x20_Pin, Connector_PinHeader_2.54mm:PinHeader_1x20_P2.54mm_Vertical, symbol Connector:Conn_01x20_Pin
- added C1, C2, C3: C, Capacitor_SMD:C_0805_2012Metric, symbol Device:C
- added Down1, Left1, Right1, Up1: SW_Push, Button_Switch_SMD:SW_SPST_PTS810, symbol Switch:SW_Push
- added R3, R4, R5, R6, R7, R8, R9: R, Resistor_SMD:R_0201_0603Metric, symbol Device:R
- renumbered Down1 to Bottom_button1, OnOff to OnOff1, UP1 to Top_button1
Connections:
- net A1: now also 01-GND_Breakout1.4 (Pin_4)
- net A2: now also 01-GND_Breakout1.5 (Pin_5)
- net A3: now also 01-GND_Breakout1.6 (Pin_6)
- net A5: now also 01-GND_Breakout1.7 (Pin_7)
- net Down: now also Down1.1, R4.2; no longer Bottom_button1.1, DevBoardI01-GND1.2 (Pin_2)
- net GND: now also 01-GND_Breakout1.20 (Pin_20), 46-GND_Breakout1.20 (Pin_20), C1.1, C2.1, C3.2, R7.1, R8.1, R9.1; no longer Bottom_button1.2, Select1.2, Top_button1.2
- net SD1: now also 01-GND_Breakout1.10 (Pin_10)
- net SD2: now also 01-GND_Breakout1.11 (Pin_11)
- net SD3: now also 01-GND_Breakout1.12 (Pin_12)
- net SD4: now also 01-GND_Breakout1.13 (Pin_13)
- net Select: now also 01-GND_Breakout1.8 (Pin_8), R8.2
- net Up: now also R3.2, Up1.1; no longer DevBoardI01-GND1.1 (Pin_1), Top_button1.1
- net Vin(3.3): now also Bottom_button1.2, Select1.2, Top_button1.2, 01-GND_Breakout1.19 (Pin_19), Down1.2, Left1.2, Right1.2, Up1.2
- net Vin(5): now also 46-GND_Breakout1.19 (Pin_19)
- net at DevBoardIO46-GND1.1 (Pin_1): now also 46-GND_Breakout1.1 (Pin_1)
- net at DevBoardIO46-GND1.10 (Pin_10): now also 46-GND_Breakout1.10 (Pin_10)
- net at DevBoardIO46-GND1.11 (Pin_11): now also 46-GND_Breakout1.11 (Pin_11)
- net at DevBoardIO46-GND1.12 (Pin_12): now also 46-GND_Breakout1.12 (Pin_12)
- net at DevBoardIO46-GND1.13 (Pin_13): now also 46-GND_Breakout1.13 (Pin_13)
- net at DevBoardIO46-GND1.14 (Pin_14): now also 46-GND_Breakout1.14 (Pin_14)
- net at DevBoardIO46-GND1.15 (Pin_15): now also 46-GND_Breakout1.15 (Pin_15)
- net at DevBoardIO46-GND1.16 (Pin_16): now also 46-GND_Breakout1.16 (Pin_16)
- net at DevBoardIO46-GND1.17 (Pin_17): now also 46-GND_Breakout1.17 (Pin_17)
- net at DevBoardIO46-GND1.18 (Pin_18): now also 46-GND_Breakout1.18 (Pin_18)
- net at DevBoardIO46-GND1.2 (Pin_2): now also 46-GND_Breakout1.2 (Pin_2)
- net at DevBoardIO46-GND1.3 (Pin_3): now also 46-GND_Breakout1.3 (Pin_3)
- net at DevBoardIO46-GND1.4 (Pin_4): now also 46-GND_Breakout1.4 (Pin_4)
- net at DevBoardIO46-GND1.5 (Pin_5): now also 46-GND_Breakout1.5 (Pin_5)
- net at DevBoardIO46-GND1.6 (Pin_6): now also 46-GND_Breakout1.6 (Pin_6)
- net at DevBoardIO46-GND1.7 (Pin_7): now also 46-GND_Breakout1.7 (Pin_7)
- net at DevBoardIO46-GND1.8 (Pin_8): now also 46-GND_Breakout1.8 (Pin_8)
- net at DevBoardIO46-GND1.9 (Pin_9): now also 46-GND_Breakout1.9 (Pin_9)
- net at DevBoardI01-GND1.14 (Pin_14): now also 01-GND_Breakout1.14 (Pin_14)
- net at DevBoardI01-GND1.15 (Pin_15): now also 01-GND_Breakout1.15 (Pin_15)
- net D-Pad_in: now reaches DevBoardI01-GND1.16 (Pin_16)
- net D-Pad_in: now also 01-GND_Breakout1.16 (Pin_16), C1.2, C2.2, C3.1, R3.1, R4.1, R5.1, R6.1
- net at DevBoardI01-GND1.17 (Pin_17): now also 01-GND_Breakout1.17 (Pin_17)
- net at DevBoardI01-GND1.18 (Pin_18): now also 01-GND_Breakout1.18 (Pin_18)
- net at DevBoardI01-GND1.3 (Pin_3): now also 01-GND_Breakout1.3 (Pin_3)
- net at DevBoardI01-GND1.9 (Pin_9): now also 01-GND_Breakout1.9 (Pin_9)
- new net Bottom: 01-GND_Breakout1.2 (Pin_2), Bottom_button1.1, DevBoardI01-GND1.2 (Pin_2), R9.2
- new net Left: Left1.1, R5.2
- new net Right: R6.2, Right1.1
- new net Top: 01-GND_Breakout1.1 (Pin_1), DevBoardI01-GND1.1 (Pin_1), R7.2, Top_button1.1
- no-connect marks 0 -> 1
Other:
- note added: "D-Pad Resistor Tree"
- note added: "D-pad Buttons"
- note added: "Selection Buttons"
- moved on the sheet: Amplifier1, Bottom_button1, DevBoardI01-GND1, DevBoardIO46-GND1, PathToGND1, PathToVin1, R1, R2, SDAdaptor1, Select1, Top_button1

Commit message: Kicad Work
Parts:
- added C4, C5, C6: C, Capacitor_SMD:C_0805_2012Metric, symbol Device:C
Connections:
- net Bottom: now also C6.1
- net GND: now also C4.2, C5.2, C6.2
- net Select: now also C4.1
- net Top: now also C5.1
Other:
- moved on the sheet: R7, Top_button1

Commit message: current Kicad
Parts:
- added C4: C, Capacitor_SMD:C_0805_2012Metric, symbol Device:C
- renumbered C4 to C7
Connections:
- net D-Pad_in: no longer C1.2, C2.2, C3.1, R3.1, R4.1, R5.1, R6.1
- net GND: now also C1.2, C2.2, R3.1, R4.1, R5.1, R6.1, C4.2; no longer C1.1, C2.1
- net Down renamed D-Pad_Down
- net D-Pad_Down: now also C3.1
- net Left renamed D-Pad_Left
- net D-Pad_Left: now also C2.1
- net Right renamed D-Pad_Right
- net D-Pad_Right: now also C1.1
- net Up renamed D-Pad_Up
- net D-Pad_Up: now also C4.1
Other:
- note added: "D-Pad C/R Tree"
- note removed: "D-Pad Resistor Tree"
- company: (none) -> Brain Buddies
- title: (none) -> Brain Buddies Assistive Device
- moved on the sheet: Bottom_button1, C1, C2, C3, C6, C7, R3, R4, R5, R6, R8, R9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

Commit message: Last nov 3 update
Connections:
- net D-Pad_in is gone; now on net D-Pad_Down: 01-GND_Breakout1.16 (Pin_16), DevBoardI01-GND1.16 (Pin_16)
- net D-Pad_Left: now also 01-GND_Breakout1.17 (Pin_17), DevBoardI01-GND1.17 (Pin_17)
- net D-Pad_Right: now also 01-GND_Breakout1.18 (Pin_18), DevBoardI01-GND1.18 (Pin_18)
- net D-Pad_Up: now also 01-GND_Breakout1.15 (Pin_15), DevBoardI01-GND1.15 (Pin_15)
Other:
- note added: "TODO: Check LCD pin assignment •Finish Boking and labeling •Check that buttons are set correctly"
- moved on the sheet: C1, C2, C3, C4, R3, R4, R5, R6

Commit message: pcb Edits
Parts:
- renumbered C4 to C3, C3 to C4, C2 to C5, C1 to C6, C5 to C7, C7 to C8, C6 to C9
Connections:
- net - is gone; now on net GND: GenConnector1.1 (Pin_1), JSTBattery1.1 (Pin_1)

Commit message: Current KiCAD November 4 5PM
Parts:
- C3, C4, C5, C6, C7, C8, C9: footprint Capacitor_SMD:C_0805_2012Metric -> Capacitor_SMD:C_0805_2012Metric_Pad1.18x1.45mm_HandSolder
- R1, R2, R3, R4, R5, R6, R7, R8, R9: footprint Resistor_SMD:R_0201_0603Metric -> Resistor_SMD:R_0805_2012Metric_Pad1.20x1.40mm_HandSolder
Connections:
- net +: now also Amplifier1.7 (Pin_7); no longer JSTBattery1.2 (Pin_2), OnOff1.2 (B)
- net Bottom: now also 01-GND_Breakout1.3 (Pin_3), DevBoardI01-GND1.3 (Pin_3); no longer 01-GND_Breakout1.2 (Pin_2), Bottom_button1.1, DevBoardI01-GND1.2 (Pin_2)
- net D-Pad_Down: now also 01-GND_Breakout1.14 (Pin_14), DevBoardI01-GND1.14 (Pin_14); no longer 01-GND_Breakout1.16 (Pin_16), DevBoardI01-GND1.16 (Pin_16), Down1.1
- net D-Pad_Left: now also 01-GND_Breakout1.15 (Pin_15), DevBoardI01-GND1.15 (Pin_15); no longer 01-GND_Breakout1.17 (Pin_17), DevBoardI01-GND1.17 (Pin_17), Left1.1
- net D-Pad_Right: now also 01-GND_Breakout1.16 (Pin_16), DevBoardI01-GND1.16 (Pin_16); no longer 01-GND_Breakout1.18 (Pin_18), DevBoardI01-GND1.18 (Pin_18), Right1.1
- net D-Pad_Up: now also 01-GND_Breakout1.17 (Pin_17), DevBoardI01-GND1.17 (Pin_17); no longer 01-GND_Breakout1.15 (Pin_15), DevBoardI01-GND1.15 (Pin_15), Up1.1
- net GND: no longer R3.1, R4.1, R5.1, R6.1, R7.1, R8.1, R9.1
- net Select: now also 01-GND_Breakout1.2 (Pin_2), DevBoardI01-GND1.2 (Pin_2); no longer 01-GND_Breakout1.8 (Pin_8), DevBoardI01-GND1.8 (Pin_8), Select1.1
- net Top: no longer Top_button1.1
- net Vin(3.3): no longer Amplifier1.7 (Pin_7)
- net IO46: now reaches 46-GND_Breakout1.1 (Pin_1), DevBoardIO46-GND1.1 (Pin_1)
- net IO37: now reaches 46-GND_Breakout1.10 (Pin_10), DevBoardIO46-GND1.10 (Pin_10)
- net IO36: now reaches 46-GND_Breakout1.11 (Pin_11), DevBoardIO46-GND1.11 (Pin_11)
- net IO35: now reaches 46-GND_Breakout1.12 (Pin_12), DevBoardIO46-GND1.12 (Pin_12)
- net IO48: now reaches 46-GND_Breakout1.13 (Pin_13), DevBoardIO46-GND1.13 (Pin_13)
- net IO34: now reaches 46-GND_Breakout1.14 (Pin_14), DevBoardIO46-GND1.14 (Pin_14)
- net IO33: now reaches 46-GND_Breakout1.15 (Pin_15), DevBoardIO46-GND1.15 (Pin_15)
- net IO47: now reaches 46-GND_Breakout1.16 (Pin_16), DevBoardIO46-GND1.16 (Pin_16)
- net IO26: now reaches 46-GND_Breakout1.17 (Pin_17), DevBoardIO46-GND1.17 (Pin_17)
- net IO21: now reaches 46-GND_Breakout1.18 (Pin_18), DevBoardIO46-GND1.18 (Pin_18)
- net IO45: now reaches 46-GND_Breakout1.2 (Pin_2), DevBoardIO46-GND1.2 (Pin_2)
- net RX0: now reaches 46-GND_Breakout1.3 (Pin_3), DevBoardIO46-GND1.3 (Pin_3)
- net TX0: now reaches 46-GND_Breakout1.4 (Pin_4), DevBoardIO46-GND1.4 (Pin_4)
- net IO42: now reaches 46-GND_Breakout1.5 (Pin_5), DevBoardIO46-GND1.5 (Pin_5)
- net IO41: now reaches 46-GND_Breakout1.6 (Pin_6), DevBoardIO46-GND1.6 (Pin_6)
- net IO40: now reaches 46-GND_Breakout1.7 (Pin_7), DevBoardIO46-GND1.7 (Pin_7)
- net IO39: now reaches 46-GND_Breakout1.8 (Pin_8), DevBoardIO46-GND1.8 (Pin_8)
- net IO38: now reaches 46-GND_Breakout1.9 (Pin_9), DevBoardIO46-GND1.9 (Pin_9)
- new net: 01-GND_Breakout1.18 (Pin_18), DevBoardI01-GND1.18 (Pin_18)
- new net: 01-GND_Breakout1.8 (Pin_8), DevBoardI01-GND1.8 (Pin_8)
- new net: JSTBattery1.2 (Pin_2), OnOff1.2 (B)
- new net Bottom_Button: Bottom_button1.1, R9.1
- new net Down: Down1.1, R4.1
- new net Left: Left1.1, R5.1
- new net Right: R6.1, Right1.1
- new net Select_Button: R8.1, Select1.1
- new net Top_Button: R7.1, Top_button1.1
- new net Up: R3.1, Up1.1
Other:
- note added: "Amplifier Circuit (MAX98357)"
- note added: "D-Pad Debounce"
- note added: "Micro SD Card Adapter"
- note added: "Selection Buttons Debounce"
- note added: "TODO: Check LCD pin assignment •Finish Boxing and labeling •Check that buttons are set correctly"
- note removed: "D-Pad C/R Tree"
- note removed: "TODO: Check LCD pin assignment •Finish Boking and labeling •Check that buttons are set correctly"
- moved on the sheet: 01-GND_Breakout1, 46-GND_Breakout1, Amplifier1, Bottom_button1, C3, C4, C5, C6, DevBoardI01-GND1, DevBoardIO46-GND1, Down1, GenConnector1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

Commit message: update again
Connections:
- net D-Pad_Down: now also 01-GND_Breakout1.15 (Pin_15), DevBoardI01-GND1.15 (Pin_15); no longer 01-GND_Breakout1.14 (Pin_14), DevBoardI01-GND1.14 (Pin_14)
- net D-Pad_Left: now also 01-GND_Breakout1.17 (Pin_17), DevBoardI01-GND1.17 (Pin_17); no longer 01-GND_Breakout1.15 (Pin_15), DevBoardI01-GND1.15 (Pin_15)
- net D-Pad_Right: now also 01-GND_Breakout1.14 (Pin_14), DevBoardI01-GND1.14 (Pin_14); no longer 01-GND_Breakout1.16 (Pin_16), DevBoardI01-GND1.16 (Pin_16)
- net D-Pad_Up: now also 01-GND_Breakout1.16 (Pin_16), DevBoardI01-GND1.16 (Pin_16); no longer 01-GND_Breakout1.17 (Pin_17), DevBoardI01-GND1.17 (Pin_17)
Changed lines of the file:
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@@
 		)
 	)
-	(label "D-Pad_Right"
+	(label "D-Pad_Up"
 		(at 105.41 132.08 0)
 		(fields_autoplaced yes)
@@
 		)
 	)
-	(label "D-Pad_Up"
+	(label "D-Pad_Left"
 		(at 105.41 134.62 0)
 		(fields_autoplaced yes)
@@
 		)
 	)
-	(label "D-Pad_Left"
+	(label "D-Pad_Down"
 		(at 105.41 129.54 0)
 		(fields_autoplaced yes)
@@
 		)
 	)
-	(label "D-Pad_Down"
+	(label "D-Pad_Right"
 		(at 105.41 127 0)
 		(fields_autoplaced yes)

Commit message: LDC PCB
Parts:
- added LCD: Conn_01x14_Pin, symbol Connector:Conn_01x14_Pin
Connections:
- net GND: now also LCD.2 (Pin_2)
- net IO34: now also LCD.3 (Pin_3)
- net IO35: now also LCD.9 (Pin_9)
- net IO36: now also LCD.7 (Pin_7)
- net IO37: now also LCD.6 (Pin_6)
- net Vin(3.3): now also LCD.1 (Pin_1)
Other:
- note added: "LCD"
