File: PCB/Final_Project_PCB/Final_Project_PCB.kicad_sch (KiCad schematic)
At the start: 35 parts

Commit message: updates againnnn
Parts:
- LCD1: renamed from LCD; footprint (none) -> Connector_PinHeader_2.54mm:PinHeader_1x14_P2.54mm_Vertical
Connections:
- net IO33: now also LCD1.4 (Pin_4)
- net IO41: now also LCD1.8 (Pin_8)
- net IO42: now also LCD1.10 (Pin_10)
- net IO45: now also LCD1.13 (Pin_13)
- net IO46: now also LCD1.14 (Pin_14)
- net IO47: now also LCD1.5 (Pin_5)
- net IO43: now reaches LCD1.11 (Pin_11)
- net IO44: now reaches LCD1.12 (Pin_12)
Other:
- moved on the sheet: Bottom_button1, Top_button1
Changed lines of the file:
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@@
 	(wire
 		(pts
-			(xy 180.34 76.2) (xy 180.34 82.55)
+			(xy 157.48 76.2) (xy 157.48 82.55)
 		)
 		(stroke
@@
 	(wire
 		(pts
-			(xy 157.48 76.2) (xy 157.48 82.55)
+			(xy 180.34 76.2) (xy 180.34 82.55)
 		)
 		(stroke
@@
 	(wire
 		(pts
+			(xy 170.18 76.2) (xy 170.18 82.55)
+		)
+		(stroke
+			(width 0)
+			(type default)
+		)
+	)
+	(wire
+		(pts
 			(xy 64.77 26.67) (xy 64.77 38.1)
 		)
@@
 	(wire
 		(pts
-			(xy 160.02 76.2) (xy 160.02 82.55)
-		)
-		(stroke
-			(width 0)
-			(type default)
-		)
-	)
-	(wire
-		(pts
 			(xy 41.91 111.76) (xy 59.69 111.76)
 		)
@@
 	(wire
 		(pts
-			(xy 170.18 76.2) (xy 170.18 82.55)
-		)
-		(stroke
-			(width 0)
-			(type default)
-		)
-	)
-	(wire
-		(pts
 			(xy 97.79 134.62) (xy 123.19 134.62)
 		)
@@
 	(wire
 		(pts
-			(xy 222.25 54.61) (xy 229.87 54.61)
+			(xy 227.33 54.61) (xy 234.95 54.61)
 		)
 		(stroke
@@
 	(wire
 		(pts
-			(xy 162.56 76.2) (xy 162.56 82.55)
+			(xy 154.94 49.53) (xy 170.18 49.53)
 		)
 		(stroke
@@
 	(wire
 		(pts
-			(xy 154.94 49.53) (xy 170.18 49.53)
+			(xy 97.79 109.22) (xy 123.19 109.22)
 		)
 		(stroke
@@
 	(wire
 		(pts
-			(xy 97.79 109.22) (xy 123.19 109.22)
+			(xy 162.56 76.2) (xy 162.56 82.55)
 		)
 		(stroke
@@
 	(wire
 		(pts
+			(xy 160.02 76.2) (xy 160.02 82.55)
+		)
+		(stroke
+			(width 0)
+			(type default)
+		)
+	)
+	(wire
+		(pts
 			(xy 214.63 148.59) (xy 224.79 148.59)
 		)
@@
 	(wire
 		(pts
-			(xy 223.52 29.21) (xy 232.41 29.21)
+			(xy 228.6 29.21) (xy 237.49 29.21)
 		)
 		(stroke
@@
 	(wire
 		(pts
-			(xy 243.84 54.61) (xy 243.84 58.42)
+			(xy 248.92 54.61) (xy 248.92 58.42)
 		)
 		(stroke
@@
 	(wire
 		(pts
-			(xy 242.57 29.21) (xy 243.84 29.21)
+			(xy 247.65 29.21) (xy 248.92 29.21)
 		)
 		(stroke
@@
 	(wire
 		(pts
-			(xy 243.84 29.21) (xy 243.84 33.02)
+			(xy 248.92 29.21) (xy 248.92 33.02)
 		)
 		(stroke
@@
 	(wire
 		(pts
-			(xy 240.03 54.61) (xy 243.84 54.61)
+			(xy 245.11 54.61) (xy 248.92 54.61)
 		)
 		(stroke
@@
 	)
 	(label "IO37"
-		(at 170.18 81.28 90)
+		(at 170.18 76.2 90)
 		(fields_autoplaced yes)
 		(effects
@@
 		)
 	)
+	(label "IO47"
+		(at 167.64 76.2 90)
+		(fields_autoplaced yes)
+		(effects
+			(font
+				(size 1.27 1.27)
+			)
+			(justify left bottom)
+		)
+	)
 	(label "D-Pad_Left"
 		(at 160.02 132.08 180)
@@
 	)
 	(label "GND"
-		(at 160.02 81.28 90)
+		(at 160.02 76.2 90)
 		(fields_autoplaced yes)
 		(effects
@@
 		)
 	)
+	(label "IO33"
+		(at 165.1 76.2 90)
+		(fields_autoplaced yes)
+		(effects
+			(font
+				(size 1.27 1.27)
+			)
+			(justify left bottom)
+		)
+	)
 	(label "SD4"
 		(at 105.41 124.46 0)
@@
 	)
 	(label "Bottom_Button"
-		(at 222.25 54.61 180)
+		(at 227.33 54.61 180)
 		(fields_autoplaced yes)
 		(effects
@@
 		)
 	)
+	(label "IO46"
+		(at 190.5 76.2 90)
+		(fields_autoplaced yes)
+		(effects
+			(font
+				(size 1.27 1.27)
+			)
+			(justify left bottom)
+		)
+	)
 	(label "Vin(3.3)"
 		(at 64.77 52.07 0)
@@
 	)
 	(label "Top_Button"
-		(at 223.52 29.21 180)
+		(at 228.6 29.21 180)
 		(fields_autoplaced yes)
 		(effects
@@
 	)
 	(label "IO36"
-		(at 172.72 81.28 90)
+		(at 172.72 76.2 90)
 		(fields_autoplaced yes)
 		(effects
@@
 		)
 	)
+	(label "IO43"
+		(at 182.88 76.2 90)
+		(fields_autoplaced yes)
+		(effects
+			(font
+				(size 1.27 1.27)
+			)
+			(justify left bottom)
+		)
+	)
 	(label "Up"
 		(at 198.12 109.22 0)
@@
 		)
 	)
+	(label "IO42"
+		(at 180.34 76.2 90)
+		(fields_autoplaced yes)
+		(effects
+			(font
+				(size 1.27 1.27)
+			)
+			(justify left bottom)
+		)
+	)
 	(label "IO35"
 		(at 46.99 121.92 0)
@@
 	)
 	(label "Vin(3.3)"
-		(at 157.48 81.28 90)
+		(at 157.48 76.2 90)
 		(fields_autoplaced yes)
 		(effects
@@
 	)
 	(label "Vin(5)"
-		(at 50.8 139.7 180)
+		(at 46.99 139.7 0)
 		(fields_autoplaced yes)
 		(effects
@@
 				(size 1.27 1.27)
 			)
-			(justify right bottom)
+			(justify left bottom)
 		)
 	)
 	(label "Vin(3.3)"
-		(at 243.84 58.42 180)
+		(at 248.92 58.42 180)
 		(fields_autoplaced yes)
 		(effects
@@
 	)
 	(label "IO35"
-		(at 177.8 81.28 90)
+		(at 177.8 76.2 90)
 		(fields_autoplaced yes)
 		(effects
@@
 		)
 	)
+	(label "IO41"
+		(at 175.26 76.2 90)
+		(fields_autoplaced yes)
+		(effects
+			(font
+				(size 1.27 1.27)
+			)
+			(justify left bottom)
+		)
+	)
 	(label "Select_Button"
 		(at 254 41.91 180)
@@
 	)
 	(label "IO34"
-		(at 162.56 81.28 90)
+		(at 162.56 76.2 90)
 		(fields_autoplaced yes)
 		(effects
@@
 		)
 	)
+	(label "IO44"
+		(at 185.42 76.2 90)
+		(fields_autoplaced yes)
+		(effects
+			(font
+				(size 1.27 1.27)
+			)
+			(justify left bottom)
+		)
+	)
 	(label "IO45"
 		(at 46.99 96.52 0)
@@
 		)
 	)
+	(label "IO45"
+		(at 187.96 76.2 90)
+		(fields_autoplaced yes)
+		(effects
+			(font
+				(size 1.27 1.27)
+			)
+			(justify left bottom)
+		)
+	)
 	(label "Vin(3.3)"
 		(at 240.03 85.09 180)
@@
 	)
 	(label "Vin(3.3)"
-		(at 243.84 33.02 180)
+		(at 248.92 33.02 180)
 		(fields_autoplaced yes)
 		(effects
@@
 	(symbol
 		(lib_id "Switch:SW_Push")
-		(at 234.95 54.61 0)
+		(at 240.03 54.61 0)
 		(unit 1)
 		(exclude_from_sim no)
@@
 		(fields_autoplaced yes)
 		(property "Reference" "Bottom_button1"
-			(at 234.95 46.99 0)
+			(at 240.03 46.99 0)
 			(effects
 				(font
@@
 		)
 		(property "Value" "SW_Push"
-			(at 234.95 49.53 0)
+			(at 240.03 49.53 0)
 			(effects
 				(font
@@
 		)
 		(property "Footprint" "Button_Switch_SMD:SW_SPST_PTS810"
-			(at 234.95 49.53 0)
+			(at 240.03 49.53 0)
 			(effects
 				(font
@@
 		)
 		(property "Datasheet" "~"
-			(at 234.95 49.53 0)
+			(at 240.03 49.53 0)
 			(effects
 				(font
@@
 		)
 		(property "Description" "Push button switch, generic, two pins"
-			(at 234.95 54.61 0)
+			(at 240.03 54.61 0)
 			(effects
 				(font
@@
 		(dnp no)
 		(fields_autoplaced yes)
-		(property "Reference" "LCD"
+		(property "Reference" "LCD1"
 			(at 173.99 90.17 90)
 			(effects
@@
 			)
 		)
-		(property "Footprint" ""
+		(property "Footprint" "Connector_PinHeader_2.54mm:PinHeader_1x14_P2.54mm_Vertical"
 			(at 172.72 87.63 0)
 			(effects
@@
 			(project ""
 				(path "/539b41c1-4420-4cfd-92b7-a29c74941d81"
-					(reference "LCD")
+					(reference "LCD1")
 					(unit 1)
 				)
@@
 	(symbol
 		(lib_id "Switch:SW_Push")
-		(at 237.49 29.21 0)
+		(at 242.57 29.21 0)
 		(unit 1)
 		(exclude_from_sim no)
@@
 		(fields_autoplaced yes)
 		(property "Reference" "Top_button1"
-			(at 237.49 21.59 0)
+			(at 242.57 21.59 0)
 			(effects
 				(font
@@
 		)
 		(property "Value" "SW_Push"
-			(at 237.49 24.13 0)
+			(at 242.57 24.13 0)
 			(effects
 				(font
@@
 		)
 		(property "Footprint" "Button_Switch_SMD:SW_SPST_PTS810"
-			(at 237.49 24.13 0)
+			(at 242.57 24.13 0)
 			(effects
 				(font
@@
 		)
 		(property "Datasheet" "~"
-			(at 237.49 24.13 0)
+			(at 242.57 24.13 0)
 			(effects
 				(font
@@
 		)
 		(property "Description" "Push button switch, generic, two pins"
-			(at 237.49 29.21 0)
+			(at 242.57 29.21 0)
 			(effects
 				(font

Commit message: Save before filling in front and back planes with copper
Parts:
- removed OnOff1: SW_SPDT, Button_Switch_SMD:SW_SPDT_CK_JS102011SAQN, symbol Switch:SW_SPDT
- added SS1: SW_Slide_DPDT, Button_Switch_SMD:SW_DPDT_CK_JS202011JCQN, symbol Switch:SW_Slide_DPDT
Connections:
- net RX0 is gone; now on net IO44: 46-GND_Breakout1.3 (Pin_3), DevBoardIO46-GND1.3 (Pin_3)
- net TX0 is gone; now on net IO43: 46-GND_Breakout1.4 (Pin_4), DevBoardIO46-GND1.4 (Pin_4)
- net +: now also SS1.1 (A), SS1.4 (A)
- net at JSTBattery1.2 (Pin_2): now also SS1.2 (B), SS1.5 (B)
- no-connect marks 1 -> 2
Other:
- moved on the sheet: JSTBattery1
Changed lines of the file:
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@@
 	)
 	(junction
+		(at 72.39 151.13)
+		(diameter 0)
+		(color 0 0 0 0)
+	)
+	(junction
 		(at 107.95 142.24)
 		(diameter 0)
@@
 	)
 	(junction
+		(at 76.2 163.83)
+		(diameter 0)
+		(color 0 0 0 0)
+	)
+	(junction
 		(at 176.53 109.22)
 		(diameter 0)
@@
 	)
 	(no_connect
-		(at 76.2 153.67)
+		(at 71.12 153.67)
+	)
+	(no_connect
+		(at 81.28 163.83)
 	)
 	(wire
@@
 	(wire
 		(pts
+			(xy 81.28 153.67) (xy 81.28 151.13)
+		)
+		(stroke
+			(width 0)
+			(type default)
+		)
+	)
+	(wire
+		(pts
 			(xy 237.49 148.59) (xy 237.49 152.4)
 		)
@@
 	(wire
 		(pts
-			(xy 71.12 148.59) (xy 71.12 153.67)
+			(xy 33.02 44.45) (xy 33.02 26.67)
 		)
 		(stroke
@@
 	(wire
 		(pts
-			(xy 33.02 44.45) (xy 33.02 26.67)
+			(xy 72.39 151.13) (xy 72.39 148.59)
 		)
 		(stroke
@@
 	(wire
 		(pts
+			(xy 71.12 163.83) (xy 64.77 163.83)
+		)
+		(stroke
+			(width 0)
+			(type default)
+		)
+	)
+	(wire
+		(pts
 			(xy 154.94 49.53) (xy 170.18 49.53)
 		)
@@
 	(wire
 		(pts
-			(xy 73.66 148.59) (xy 71.12 148.59)
+			(xy 73.66 148.59) (xy 72.39 148.59)
 		)
 		(stroke
@@
 	(wire
 		(pts
+			(xy 64.77 151.13) (xy 72.39 151.13)
+		)
+		(stroke
+			(width 0)
+			(type default)
+		)
+	)
+	(wire
+		(pts
 			(xy 41.91 109.22) (xy 59.69 109.22)
 		)
@@
 	(wire
 		(pts
-			(xy 73.66 163.83) (xy 73.66 176.53)
+			(xy 76.2 163.83) (xy 76.2 176.53)
 		)
 		(stroke
@@
 	(wire
 		(pts
+			(xy 64.77 163.83) (xy 64.77 151.13)
+		)
+		(stroke
+			(width 0)
+			(type default)
+		)
+	)
+	(wire
+		(pts
 			(xy 97.79 99.06) (xy 123.19 99.06)
 		)
@@
 	(wire
 		(pts
-			(xy 58.42 176.53) (xy 73.66 176.53)
+			(xy 60.96 176.53) (xy 76.2 176.53)
 		)
 		(stroke
@@
 	(wire
 		(pts
+			(xy 76.2 153.67) (xy 76.2 163.83)
+		)
+		(stroke
+			(width 0)
+			(type default)
+		)
+	)
+	(wire
+		(pts
 			(xy 160.02 132.08) (xy 176.53 132.08)
 		)
@@
 	(wire
 		(pts
-			(xy 58.42 173.99) (xy 67.31 173.99)
+			(xy 60.96 173.99) (xy 69.85 173.99)
 		)
 		(stroke
@@
 	(wire
 		(pts
+			(xy 81.28 151.13) (xy 72.39 151.13)
+		)
+		(stroke
+			(width 0)
+			(type default)
+		)
+	)
+	(wire
+		(pts
 			(xy 254 41.91) (xy 262.89 41.91)
 		)
@@
 		)
 	)
-	(label "TX0"
+	(label "IO43"
 		(at 46.99 101.6 0)
 		(fields_autoplaced yes)
@@
 		)
 	)
-	(label "RX0"
+	(label "IO44"
 		(at 46.99 99.06 0)
 		(fields_autoplaced yes)
@@
 	)
 	(label "-"
-		(at 60.96 173.99 0)
+		(at 63.5 173.99 0)
 		(fields_autoplaced yes)
 		(effects
@@
 	(symbol
 		(lib_id "power:GND")
-		(at 67.31 173.99 180)
+		(at 69.85 173.99 180)
 		(unit 1)
 		(exclude_from_sim no)
@@
 		(fields_autoplaced yes)
 		(property "Reference" "#PWR015"
-			(at 67.31 167.64 0)
+			(at 69.85 167.64 0)
 			(effects
 				(font
@@
 		)
 		(property "Value" "GND"
-			(at 67.31 168.91 0)
+			(at 69.85 168.91 0)
 			(effects
 				(font
@@
 		)
 		(property "Footprint" ""
-			(at 67.31 173.99 0)
+			(at 69.85 173.99 0)
 			(effects
 				(font
@@
 		)
 		(property "Datasheet" ""
-			(at 67.31 173.99 0)
+			(at 69.85 173.99 0)
 			(effects
 				(font
@@
 		)
 		(property "Description" "Power symbol creates a global label with name \"GND\" , ground"
-			(at 67.31 173.99 0)
+			(at 69.85 173.99 0)
 			(effects
 				(font
@@
 	(symbol
 		(lib_id "Connector:Conn_01x02_Pin")
-		(at 53.34 173.99 0)
+		(at 55.88 173.99 0)
 		(unit 1)
 		(exclude_from_sim no)
@@
 		(fields_autoplaced yes)
 		(property "Reference" "JSTBattery1"
-			(at 53.975 168.91 0)
+			(at 56.515 168.91 0)
 			(effects
 				(font
@@
 		)
 		(property "Value" "Conn_01x02_Pin"
-			(at 53.975 171.45 0)
+			(at 56.515 171.45 0)
 			(effects
 				(font
@@
 		)
 		(property "Footprint" "Connector_JST:JST_PH_S2B-PH-K_1x02_P2.00mm_Horizontal"
-			(at 53.34 173.99 0)
+			(at 55.88 173.99 0)
 			(effects
 				(font
@@
 		)
 		(property "Datasheet" "~"
-			(at 53.34 173.99 0)
+			(at 55.88 173.99 0)
 			(effects
 				(font
@@
 		)
 		(property "Description" "Generic connector, single row, 01x02, script generated"
-			(at 53.34 173.99 0)
+			(at 55.88 173.99 0)
 			(effects
 				(font
@@
 	)
 	(symbol
-		(lib_id "Device:R")
-		(at 118.11 41.91 0)
+		(lib_id "Switch:SW_Slide_DPDT")
+		(at 76.2 158.75 90)
 		(unit 1)
 		(exclude_from_sim no)
@@
 		(on_board yes)
 		(dnp no)
-		(fields_autoplaced yes)
-		(property "Reference" "R1"
-			(at 120.65 40.6399 0)
+		(property "Reference" "SS1"
+			(at 66.04 158.75 0)
 			(effects
 				(font
 					(size 1.27 1.27)
 				)
-				(justify left)
 			)
 		)
-		(property "Value" "100k"
-			(at 120.65 43.1799 0)
+		(property "Value" "SW_Slide_DPDT"
+			(at 68.58 158.75 0)
 			(effects
 				(font
 					(size 1.27 1.27)
 				)
-				(justify left)
 			)
 		)
-		(property "Footprint" "Resistor_SMD:R_0805_2012Metric_Pad1.20x1.40mm_HandSolder"
-			(at 116.332 41.91 90)
+		(property "Footprint" "Button_Switch_SMD:SW_DPDT_CK_JS202011JCQN"
+			(at 71.12 144.78 0)
 			(effects
 				(font
@@
 		)
 		(property "Datasheet" "~"
-			(at 118.11 41.91 0)
+			(at 76.2 158.75 0)
 			(effects
 				(font
@@
 			)
 		)
-		(property "Description" "Resistor"
-			(at 118.11 41.91 0)
+		(property "Description" "Slide Switch, dual pole double throw"
+			(at 76.2 158.75 0)
 			(effects
 				(font
@@
 			)
 		)
+		(pin "2"
+		)
+		(pin "5"
+		)
 		(pin "1"
 		)
-		(pin "2"
+		(pin "4"
+		)
+		(pin "6"
+		)
+		(pin "3"
 		)
 		(instances
 			(project ""
 				(path "/539b41c1-4420-4cfd-92b7-a29c74941d81"
-					(reference "R1")
+					(reference "SS1")
 					(unit 1)
 				)
@@
 	)
 	(symbol
-		(lib_id "Switch:SW_SPDT")
-		(at 73.66 158.75 90)
+		(lib_id "Device:R")
+		(at 118.11 41.91 0)
 		(unit 1)
 		(exclude_from_sim no)
@@
 		(on_board yes)
 		(dnp no)
-		(property "Reference" "OnOff1"
-			(at 68.58 160.0201 90)
+		(fields_autoplaced yes)
+		(property "Reference" "R1"
+			(at 120.65 40.6399 0)
 			(effects
 				(font
@@
 			)
 		)
-		(property "Value" "SW_SPDT"
-			(at 68.58 157.4801 90)
+		(property "Value" "100k"
+			(at 120.65 43.1799 0)
 			(effects
 				(font
@@
 			)
 		)
-		(property "Footprint" "Button_Switch_SMD:SW_SPDT_CK_JS102011SAQN"
-			(at 73.66 158.75 0)
+		(property "Footprint" "Resistor_SMD:R_0805_2012Metric_Pad1.20x1.40mm_HandSolder"
+			(at 116.332 41.91 90)
 			(effects
 				(font
@@
 		)
 		(property "Datasheet" "~"
-			(at 81.28 158.75 0)
+			(at 118.11 41.91 0)
 			(effects
 				(font
@@
 			)
 		)
-		(property "Description" "Switch, single pole double throw"
-			(at 73.66 158.75 0)
+		(property "Description" "Resistor"
+			(at 118.11 41.91 0)
 			(effects
 				(font
@@
 			)
 		)
-		(pin "2"
-		)
 		(pin "1"
 		)
-		(pin "3"
+		(pin "2"
 		)
 		(instances
 			(project ""
 				(path "/539b41c1-4420-4cfd-92b7-a29c74941d81"
-					(reference "OnOff1")
+					(reference "R1")
 					(unit 1)
 				)

Commit message: Final PCB Update - Pending Review
Parts:
- renumbered GenConnector1 to BatToBoard1
Connections:
- net +: now also LCD1.1 (Pin_1)
- net Vin(3.3): no longer LCD1.1 (Pin_1)
Other:
- note removed: "TODO: Check LCD pin assignment •Finish Boxing and labeling •Check that buttons are set correctly"
Changed lines of the file:
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@@
 	(title_block
 		(title "Brain Buddies Assistive Device")
-		(date "2024-11-03")
-		(rev "0")
+		(date "2024-11-04")
+		(rev "1.0")
 		(company "Brain Buddies")
 		(comment 2 "Dustin Miller")
@@
 		)
 	)
-	(text "TODO: Check LCD pin assignment •Finish Boxing and labeling •Check that buttons are set correctly"
-		(exclude_from_sim no)
-		(at 80.772 73.152 0)
-		(effects
-			(font
-				(size 1.27 1.27)
-			)
-		)
-	)
 	(text "Selection Buttons Debounce"
 		(exclude_from_sim no)
@@
 		)
 	)
-	(label "-"
-		(at 63.5 173.99 0)
-		(fields_autoplaced yes)
-		(effects
-			(font
-				(size 1.27 1.27)
-			)
-			(justify left bottom)
-		)
-	)
 	(label "Vin(3.3)"
 		(at 273.05 153.67 180)
@@
 		)
 	)
-	(label "Vin(3.3)"
+	(label "+"
 		(at 157.48 76.2 90)
 		(fields_autoplaced yes)
@@
 			)
 			(justify right bottom)
-		)
-	)
-	(label "-"
-		(at 76.2 144.78 0)
-		(fields_autoplaced yes)
-		(effects
-			(font
-				(size 1.27 1.27)
-			)
-			(justify left bottom)
 		)
 	)
@@
 		(on_board yes)
 		(dnp no)
-		(property "Reference" "GenConnector1"
+		(property "Reference" "BatToBoard1"
 			(at 77.47 135.2549 90)
 			(effects
@@
 			(project ""
 				(path "/539b41c1-4420-4cfd-92b7-a29c74941d81"
-					(reference "GenConnector1")
+					(reference "BatToBoard1")
 					(unit 1)
 				)
