File: PCB/Final_Project_PCB/Final_Project_PCB.kicad_pcb (KiCad board)
At the start: 2 copper layers, 14 parts

Commit message: Schematic Finished
Parts:
- added 01-GND_Breakout1: Conn_01x20_Pin, Connector_PinHeader_2.54mm:PinHeader_1x20_P2.54mm_Vertical, F.Cu at (98.3, 136.7)
- added 46-GND_Breakout1: Conn_01x20_Pin, Connector_PinHeader_2.54mm:PinHeader_1x20_P2.54mm_Vertical, F.Cu at (103.0, 136.7)
- added C1: C, Capacitor_SMD:C_0805_2012Metric, F.Cu at (107.5, 135.9)
- added C2: C, Capacitor_SMD:C_0805_2012Metric, F.Cu at (107.5, 138.9)
- added C3: C, Capacitor_SMD:C_0805_2012Metric, F.Cu at (107.5, 141.9)
- added Down1: SW_Push, Button_Switch_SMD:SW_SPST_PTS810, F.Cu at (50.9, 146.2)
- added Left1: SW_Push, Button_Switch_SMD:SW_SPST_PTS810, F.Cu at (50.9, 150.9)
- added R3: R, Resistor_SMD:R_0201_0603Metric, F.Cu at (55.5, 144.7)
- added R4: R, Resistor_SMD:R_0201_0603Metric, F.Cu at (55.5, 146.4)
- added R5: R, Resistor_SMD:R_0201_0603Metric, F.Cu at (55.5, 148.2)
- added R6: R, Resistor_SMD:R_0201_0603Metric, F.Cu at (55.5, 149.9)
- added R7: R, Resistor_SMD:R_0201_0603Metric, F.Cu at (106.5, 144.3)
- added R8: R, Resistor_SMD:R_0201_0603Metric, F.Cu at (106.5, 146.1)
- added R9: R, Resistor_SMD:R_0201_0603Metric, F.Cu at (106.5, 147.8)
- added Right1: SW_Push, Button_Switch_SMD:SW_SPST_PTS810, F.Cu at (50.9, 155.7)
- added Up1: SW_Push, Button_Switch_SMD:SW_SPST_PTS810, F.Cu at (50.9, 160.4)
- renumbered Down1 to Bottom_button1, UP1 to Top_button1
Connections:
- net /Down renamed /Bottom
- net /Up renamed /Top
- Bottom_button1 pad 2: /GND -> /Vin(3.3)
- DevBoardI01-GND1 pad 14: unconnected-(DevBoardI01-GND1-Pin_14-Pad14) -> Net-(01-GND_Breakout1-Pin_14)
- DevBoardI01-GND1 pad 15: unconnected-(DevBoardI01-GND1-Pin_15-Pad15) -> Net-(01-GND_Breakout1-Pin_15)
- DevBoardI01-GND1 pad 16: unconnected-(DevBoardI01-GND1-Pin_16-Pad16) -> /D-Pad_in
- DevBoardI01-GND1 pad 17: unconnected-(DevBoardI01-GND1-Pin_17-Pad17) -> Net-(01-GND_Breakout1-Pin_17)
- DevBoardI01-GND1 pad 18: unconnected-(DevBoardI01-GND1-Pin_18-Pad18) -> Net-(01-GND_Breakout1-Pin_18)
- DevBoardI01-GND1 pad 3: unconnected-(DevBoardI01-GND1-Pin_3-Pad3) -> Net-(01-GND_Breakout1-Pin_3)
- DevBoardI01-GND1 pad 9: unconnected-(DevBoardI01-GND1-Pin_9-Pad9) -> Net-(01-GND_Breakout1-Pin_9)
- DevBoardIO46-GND1 pad 1: unconnected-(DevBoardIO46-GND1-Pin_1-Pad1) -> Net-(46-GND_Breakout1-Pin_1)
- DevBoardIO46-GND1 pad 10: unconnected-(DevBoardIO46-GND1-Pin_10-Pad10) -> Net-(46-GND_Breakout1-Pin_10)
- DevBoardIO46-GND1 pad 11: unconnected-(DevBoardIO46-GND1-Pin_11-Pad11) -> Net-(46-GND_Breakout1-Pin_11)
- DevBoardIO46-GND1 pad 12: unconnected-(DevBoardIO46-GND1-Pin_12-Pad12) -> Net-(46-GND_Breakout1-Pin_12)
- DevBoardIO46-GND1 pad 13: unconnected-(DevBoardIO46-GND1-Pin_13-Pad13) -> Net-(46-GND_Breakout1-Pin_13)
- DevBoardIO46-GND1 pad 14: unconnected-(DevBoardIO46-GND1-Pin_14-Pad14) -> Net-(46-GND_Breakout1-Pin_14)
- DevBoardIO46-GND1 pad 15: unconnected-(DevBoardIO46-GND1-Pin_15-Pad15) -> Net-(46-GND_Breakout1-Pin_15)
- DevBoardIO46-GND1 pad 16: unconnected-(DevBoardIO46-GND1-Pin_16-Pad16) -> Net-(46-GND_Breakout1-Pin_16)
- DevBoardIO46-GND1 pad 17: unconnected-(DevBoardIO46-GND1-Pin_17-Pad17) -> Net-(46-GND_Breakout1-Pin_17)
- DevBoardIO46-GND1 pad 18: unconnected-(DevBoardIO46-GND1-Pin_18-Pad18) -> Net-(46-GND_Breakout1-Pin_18)
- DevBoardIO46-GND1 pad 2: unconnected-(DevBoardIO46-GND1-Pin_2-Pad2) -> Net-(46-GND_Breakout1-Pin_2)
- DevBoardIO46-GND1 pad 3: unconnected-(DevBoardIO46-GND1-Pin_3-Pad3) -> Net-(46-GND_Breakout1-Pin_3)
- DevBoardIO46-GND1 pad 4: unconnected-(DevBoardIO46-GND1-Pin_4-Pad4) -> Net-(46-GND_Breakout1-Pin_4)
- DevBoardIO46-GND1 pad 5: unconnected-(DevBoardIO46-GND1-Pin_5-Pad5) -> Net-(46-GND_Breakout1-Pin_5)
- DevBoardIO46-GND1 pad 6: unconnected-(DevBoardIO46-GND1-Pin_6-Pad6) -> Net-(46-GND_Breakout1-Pin_6)
- DevBoardIO46-GND1 pad 7: unconnected-(DevBoardIO46-GND1-Pin_7-Pad7) -> Net-(46-GND_Breakout1-Pin_7)
- DevBoardIO46-GND1 pad 8: unconnected-(DevBoardIO46-GND1-Pin_8-Pad8) -> Net-(46-GND_Breakout1-Pin_8)
- DevBoardIO46-GND1 pad 9: unconnected-(DevBoardIO46-GND1-Pin_9-Pad9) -> Net-(46-GND_Breakout1-Pin_9)
- Select1 pad 2: /GND -> /Vin(3.3)
- Top_button1 pad 2: /GND -> /Vin(3.3)

Commit message: Kicad Work
Parts:
- added C4: C, Capacitor_SMD:C_0805_2012Metric, F.Cu at (121.0, 158.5)
- added C5: C, Capacitor_SMD:C_0805_2012Metric, F.Cu at (121.0, 161.5)
- added C6: C, Capacitor_SMD:C_0805_2012Metric, F.Cu at (121.0, 164.5)
- 01-GND_Breakout1, 46-GND_Breakout1, Amplifier1, C1, C2, C3, DevBoardI01-GND1, DevBoardIO46-GND1, GenConnector1, JSTBattery1, PathToGND1, PathToVin1, R1, R2, R7, R8, R9, SDAdaptor1: moved to B.Cu
- moved Amplifier1 200.8 mm to (245.6, 103.0), turned to 90 degrees
- moved OnOff1 168.5 mm to (219.5, 147.0), turned to 0 degrees
- moved 46-GND_Breakout1 162.0 mm to (239.2, 49.0), turned to 90 degrees
- moved Right1 154.6 mm to (202.0, 123.0)
- moved 01-GND_Breakout1 150.0 mm to (239.1, 85.0), turned to 90 degrees
- moved Up1 146.9 mm to (190.9, 116.1)
- moved Down1 140.5 mm to (190.6, 130.6)
- moved Left1 133.9 mm to (182.1, 123.9)
- moved Select1 129.5 mm to (248.5, 123.0)
- moved R4 125.5 mm to (176.3, 112.5)
- moved R6 125.0 mm to (176.3, 118.0)
- moved R5 120.9 mm to (170.8, 112.0)
- moved R3 118.5 mm to (170.8, 117.5)
- moved DevBoardI01-GND1 114.3 mm to (239.1, 77.8), turned to 90 degrees
- moved SDAdaptor1 112.3 mm to (197.2, 103.0), turned to 90 degrees
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
Commit message: current Kicad
Parts:
- moved R5 14.7 mm to (175.8, 125.9), turned to 90 degrees
- moved R4 13.7 mm to (173.2, 125.9), turned to 90 degrees
- moved R3 8.38 mm to (170.6, 125.9), turned to 90 degrees
- moved R6 8.14 mm to (178.4, 125.9), turned to 90 degrees
- moved Up1 4.28 mm to (192.2, 112.0)
- moved Left1 2.24 mm to (183.1, 121.9)
- moved Down1 2.22 mm to (192.2, 132.1)
- moved Right1 1.17 mm to (201.4, 122.0)

Commit message: pcb Edits
Parts:
- added C3: C, Capacitor_SMD:C_0805_2012Metric, F.Cu at (121.0, 122.2)
- C4: renamed from C3; moved to F.Cu
- C5: renamed from C2; moved to F.Cu
- C6: renamed from C1; moved to F.Cu
- PathToGND1, PathToVin1, R1, R2, R7, R8, R9: moved to F.Cu
- moved PathToVin1 132.4 mm to (161.1, 128.1), turned to 0 degrees
- moved R2 128.9 mm to (161.2, 133.1), turned to 180 degrees
- moved R7 103.3 mm to (196.5, 126.0), turned to 90 degrees
- moved R8 102.4 mm to (196.5, 133.5), turned to 90 degrees
- moved R9 101.9 mm to (196.5, 141.0), turned to 90 degrees
- moved PathToGND1 98.1 mm to (154.7, 111.4), turned to 0 degrees
- moved R1 95.6 mm to (153.3, 123.4), turned to 180 degrees
- moved C7 87.9 mm to (201.5, 126.0), turned to -90 degrees
- moved C8 84.2 mm to (201.5, 133.5), turned to -90 degrees
- moved C9 83.8 mm to (201.5, 141.0), turned to -90 degrees
- moved R6 62.5 mm to (116.0, 129.7)
- moved Bottom_button1 61.9 mm to (178.5, 143.6)
- moved Select1 60.9 mm to (188.5, 133.6)
- moved R5 60.9 mm to (116.0, 137.2)
- moved R4 60.2 mm to (116.0, 144.7)
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- renumbered C5 to C7, C4 to C8, C6 to C9
Connections:
- 01-GND_Breakout1 pad 15: Net-(01-GND_Breakout1-Pin_15) -> /Up
- 01-GND_Breakout1 pad 16: /D-Pad_in -> /Down
- 01-GND_Breakout1 pad 17: Net-(01-GND_Breakout1-Pin_17) -> /Left
- 01-GND_Breakout1 pad 18: Net-(01-GND_Breakout1-Pin_18) -> /Right
- 01-GND_Breakout1 pad 20: /GND -> GND
- 46-GND_Breakout1 pad 20: /GND -> GND
- Amplifier1 pad 6: /GND -> GND
- C4 pad 1: /D-Pad_in -> /Down
- C4 pad 2: /GND -> GND
- C5 pad 1: /GND -> /Left
- C5 pad 2: /D-Pad_in -> GND
- C6 pad 1: /GND -> /Right
- C6 pad 2: /D-Pad_in -> GND
- C7 pad 2: /GND -> GND
- C8 pad 2: /GND -> GND
- C9 pad 2: /GND -> GND
- DevBoardI01-GND1 pad 15: Net-(01-GND_Breakout1-Pin_15) -> /Up
- DevBoardI01-GND1 pad 16: /D-Pad_in -> /Down
- DevBoardI01-GND1 pad 17: Net-(01-GND_Breakout1-Pin_17) -> /Left
- DevBoardI01-GND1 pad 18: Net-(01-GND_Breakout1-Pin_18) -> /Right
- DevBoardI01-GND1 pad 20: /GND -> GND
- DevBoardIO46-GND1 pad 20: /GND -> GND
- GenConnector1 pad 1: /- -> GND
- JSTBattery1 pad 1: /- -> GND
- PathToGND1 pad 1: /GND -> GND
- R1 pad 2: /GND -> GND
- R3 pad 1: /D-Pad_in -> GND
- R4 pad 1: /D-Pad_in -> GND
- R5 pad 1: /D-Pad_in -> GND
- R6 pad 1: /D-Pad_in -> GND
- R7 pad 1: /GND -> GND
- R8 pad 1: /GND -> GND
- R9 pad 1: /GND -> GND
- SDAdaptor1 pad 6: /GND -> GND
Routing:
- net /Right: track 0.00 -> 33.2 mm
- net /Top: track 0.00 -> 22.5 mm
- net /Up: track 0.00 -> 22.2 mm
- net /Down: track 0.00 -> 22.2 mm
- net /Bottom: track 0.00 -> 21.9 mm
- net /Left: track 0.00 -> 13.2 mm
- net /Select: track 0.00 -> 11.4 mm

Commit message: Current KiCAD November 4 5PM
Parts:
- C3, C4, C5, C6, C7, C8, C9: footprint Capacitor_SMD:C_0805_2012Metric -> Capacitor_SMD:C_0805_2012Metric_Pad1.18x1.45mm_HandSolder
- R1, R2, R3, R4, R5, R6, R7, R8, R9: footprint Resistor_SMD:R_0201_0603Metric -> Resistor_SMD:R_0805_2012Metric_Pad1.20x1.40mm_HandSolder
- moved OnOff1 110.9 mm to (255.0, 98.8), turned to 90 degrees
- moved PathToGND1 92.2 mm to (246.0, 99.2), turned to 90 degrees
- moved JSTBattery1 86.1 mm to (201.0, 61.8)
- moved PathToVin1 80.3 mm to (236.0, 99.2), turned to 90 degrees
- moved R2 73.2 mm to (226.0, 99.2), turned to -90 degrees
- moved R1 67.2 mm to (216.0, 99.2), turned to -90 degrees
- moved C9 57.9 mm to (153.7, 108.3), turned to 0 degrees
- moved R9 51.0 mm to (153.7, 113.3), turned to 180 degrees
- moved Amplifier1 50.4 mm to (188.6, 61.7)
- moved C8 49.2 mm to (159.2, 108.3), turned to 0 degrees
- moved C4 45.4 mm to (148.2, 108.3), turned to 0 degrees
- moved R4 45.0 mm to (148.2, 113.3), turned to 180 degrees
- moved R8 42.4 mm to (159.2, 113.3), turned to 180 degrees
- moved C7 40.8 mm to (164.7, 108.3), turned to 0 degrees
- moved C5 36.1 mm to (142.7, 108.3), turned to 0 degrees
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Connections:
- net Net-(46-GND_Breakout1-Pin_1) renamed /IO46
- net Net-(46-GND_Breakout1-Pin_10) renamed /IO37
- net Net-(46-GND_Breakout1-Pin_11) renamed /IO36
- net Net-(46-GND_Breakout1-Pin_12) renamed /IO35
- net Net-(46-GND_Breakout1-Pin_13) renamed /IO48
- net Net-(46-GND_Breakout1-Pin_14) renamed /IO34
- net Net-(46-GND_Breakout1-Pin_15) renamed /IO33
- net Net-(46-GND_Breakout1-Pin_16) renamed /IO47
- net Net-(46-GND_Breakout1-Pin_17) renamed /IO26
- net Net-(46-GND_Breakout1-Pin_18) renamed /IO21
- net Net-(46-GND_Breakout1-Pin_2) renamed /IO45
- net Net-(46-GND_Breakout1-Pin_3) renamed /RX0
- net Net-(46-GND_Breakout1-Pin_4) renamed /TX0
- net Net-(46-GND_Breakout1-Pin_5) renamed /IO42
- net Net-(46-GND_Breakout1-Pin_6) renamed /IO41
- net Net-(46-GND_Breakout1-Pin_7) renamed /IO40
- net Net-(46-GND_Breakout1-Pin_8) renamed /IO39
- net Net-(46-GND_Breakout1-Pin_9) renamed /IO38
- 01-GND_Breakout1 pad 14: Net-(01-GND_Breakout1-Pin_14) -> /D-Pad_Down
- 01-GND_Breakout1 pad 15: /Up -> /D-Pad_Left
- 01-GND_Breakout1 pad 16: /Down -> /D-Pad_Right
- 01-GND_Breakout1 pad 17: /Left -> /D-Pad_Up
- 01-GND_Breakout1 pad 18: /Right -> Net-(01-GND_Breakout1-Pin_18)
- 01-GND_Breakout1 pad 2: /Bottom -> /Select
- 01-GND_Breakout1 pad 3: Net-(01-GND_Breakout1-Pin_3) -> /Bottom
- 01-GND_Breakout1 pad 8: /Select -> Net-(01-GND_Breakout1-Pin_8)
- Amplifier1 pad 7: /Vin(3.3) -> /+
- Bottom_button1 pad 1: /Bottom -> /Bottom_Button
- C3 pad 1: /Up -> /D-Pad_Up
- C4 pad 1: /Down -> /D-Pad_Down
- C5 pad 1: /Left -> /D-Pad_Left
- C6 pad 1: /Right -> /D-Pad_Right
- DevBoardI01-GND1 pad 14: Net-(01-GND_Breakout1-Pin_14) -> /D-Pad_Down
- DevBoardI01-GND1 pad 15: /Up -> /D-Pad_Left
- DevBoardI01-GND1 pad 16: /Down -> /D-Pad_Right
- DevBoardI01-GND1 pad 17: /Left -> /D-Pad_Up
- DevBoardI01-GND1 pad 18: /Right -> Net-(01-GND_Breakout1-Pin_18)
- DevBoardI01-GND1 pad 2: /Bottom -> /Select
- DevBoardI01-GND1 pad 3: Net-(01-GND_Breakout1-Pin_3) -> /Bottom
- DevBoardI01-GND1 pad 8: /Select -> Net-(01-GND_Breakout1-Pin_8)
- JSTBattery1 pad 2: /+ -> Net-(JSTBattery1-Pin_2)
- OnOff1 pad 2: /+ -> Net-(JSTBattery1-Pin_2)
- R3 pad 1: GND -> /Up
- R3 pad 2: /Up -> /D-Pad_Up
- R4 pad 1: GND -> /Down
- R4 pad 2: /Down -> /D-Pad_Down
- R5 pad 1: GND -> /Left
- R5 pad 2: /Left -> /D-Pad_Left
- R6 pad 1: GND -> /Right
- R6 pad 2: /Right -> /D-Pad_Right
- R7 pad 1: GND -> /Top_Button
- R8 pad 1: GND -> /Select_Button
- R9 pad 1: GND -> /Bottom_Button
- Select1 pad 1: /Select -> /Select_Button
- Top_button1 pad 1: /Top -> /Top_Button
Routing:
- net /A1: track 0.00 -> 53.0 mm
- net /A2: track 0.00 -> 53.0 mm
- net /A3: track 0.00 -> 53.0 mm
- net /A5: track 0.00 -> 50.4 mm
- net /Right: track 33.2 -> 0.00 mm
- net /SD1: track 0.00 -> 29.1 mm
- net /SD2: track 0.00 -> 25.5 mm
- net /Top: track 22.5 -> 0.00 mm
- net /Up: track 22.2 -> 0.00 mm
- net /Down: track 22.2 -> 0.00 mm
- net /SD3: track 0.00 -> 22.1 mm
- net /Bottom: track 21.9 -> 0.00 mm
- net /SD4: track 0.00 -> 18.3 mm
- net /Left: track 13.2 -> 0.00 mm
- net /Select: track 11.4 -> 0.00 mm
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Other:
- board text added: "1500 mAh 804048 Battery"
- board text added: "2000mAh 455572 Battery"
- board text added: "ESP32-S3 DevBoard"
- board text added: "No debounce for power switch, switch to J1 and amp okay[p;k,"
- board text added: "Poth planes are ground planes"
- board text added: "put RC circuits as close to the microcontroller as possible"

Commit message: update
Parts:
- moved OnOff1 56.6 mm to (205.7, 126.6)
- moved PathToGND1 44.8 mm to (202.7, 110.7)
- moved PathToVin1 44.8 mm to (192.7, 110.7)
- moved R1 44.8 mm to (172.7, 110.7)
- moved R2 44.8 mm to (182.7, 110.7)
- moved C5 11.0 mm to (131.7, 108.3)
- moved C6 11.0 mm to (148.2, 108.3)
- moved R5 11.0 mm to (131.7, 113.3)
- moved R6 11.0 mm to (148.2, 113.3)
- moved C3 5.50 mm to (137.2, 108.3)
- moved C4 5.50 mm to (142.7, 108.3)
- moved R3 5.50 mm to (137.2, 113.3)
- moved R4 5.50 mm to (142.7, 113.3)
Changed lines of the file:
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@@
 	(footprint "Capacitor_SMD:C_0805_2012Metric_Pad1.18x1.45mm_HandSolder"
 		(layer "F.Cu")
-		(at 142.7 108.3)
+		(at 131.7 108.3)
 		(descr "Capacitor SMD 0805 (2012 Metric), square (rectangular) end terminal, IPC_7351 nominal with elongated pad for handsoldering. (Body size source: IPC-SM-782 page 76, https://www.pcb-3d.com/wordpress/wp-content/uploads/ipc-sm-782a_amendment_1_and_2.pdf, https://docs.google.com/spreadsheets/d/1BsfQQcO9C6DZCsRaXUlFlo91Tg2WpOkGARC1WS5S8t0/edit?usp=sharing), generated with kicad-footprint-generator")
 		(tags "capacitor handsolder")
@@
 	(footprint "Resistor_SMD:R_0805_2012Metric_Pad1.20x1.40mm_HandSolder"
 		(layer "F.Cu")
-		(at 216 99.2 -90)
+		(at 172.7 110.7 -90)
 		(descr "Resistor SMD 0805 (2012 Metric), square (rectangular) end terminal, IPC_7351 nominal with elongated pad for handsoldering. (Body size source: IPC-SM-782 page 72, https://www.pcb-3d.com/wordpress/wp-content/uploads/ipc-sm-782a_amendment_1_and_2.pdf), generated with kicad-footprint-generator")
 		(tags "resistor handsolder")
@@
 	(footprint "Resistor_SMD:R_0805_2012Metric_Pad1.20x1.40mm_HandSolder"
 		(layer "F.Cu")
-		(at 226 99.2 -90)
+		(at 182.7 110.7 -90)
 		(descr "Resistor SMD 0805 (2012 Metric), square (rectangular) end terminal, IPC_7351 nominal with elongated pad for handsoldering. (Body size source: IPC-SM-782 page 72, https://www.pcb-3d.com/wordpress/wp-content/uploads/ipc-sm-782a_amendment_1_and_2.pdf), generated with kicad-footprint-generator")
 		(tags "resistor handsolder")
@@
 	(footprint "Capacitor_SMD:C_0805_2012Metric_Pad1.18x1.45mm_HandSolder"
 		(layer "F.Cu")
-		(at 131.7 108.3)
+		(at 137.2 108.3)
 		(descr "Capacitor SMD 0805 (2012 Metric), square (rectangular) end terminal, IPC_7351 nominal with elongated pad for handsoldering. (Body size source: IPC-SM-782 page 76, https://www.pcb-3d.com/wordpress/wp-content/uploads/ipc-sm-782a_amendment_1_and_2.pdf, https://docs.google.com/spreadsheets/d/1BsfQQcO9C6DZCsRaXUlFlo91Tg2WpOkGARC1WS5S8t0/edit?usp=sharing), generated with kicad-footprint-generator")
 		(tags "capacitor handsolder")
@@
 	(footprint "Resistor_SMD:R_0805_2012Metric_Pad1.20x1.40mm_HandSolder"
 		(layer "F.Cu")
-		(at 142.7 113.3 180)
+		(at 131.7 113.3 180)
 		(descr "Resistor SMD 0805 (2012 Metric), square (rectangular) end terminal, IPC_7351 nominal with elongated pad for handsoldering. (Body size source: IPC-SM-782 page 72, https://www.pcb-3d.com/wordpress/wp-content/uploads/ipc-sm-782a_amendment_1_and_2.pdf), generated with kicad-footprint-generator")
 		(tags "resistor handsolder")
@@
 	(footprint "Jumper:SolderJumper-2_P1.3mm_Open_RoundedPad1.0x1.5mm"
 		(layer "F.Cu")
-		(at 236 99.2 90)
+		(at 192.7 110.7 90)
 		(descr "SMD Solder Jumper, 1x1.5mm, rounded Pads, 0.3mm gap, open")
 		(tags "solder jumper open")
@@
 	(footprint "Resistor_SMD:R_0805_2012Metric_Pad1.20x1.40mm_HandSolder"
 		(layer "F.Cu")
-		(at 131.7 113.3 180)
+		(at 137.2 113.3 180)
 		(descr "Resistor SMD 0805 (2012 Metric), square (rectangular) end terminal, IPC_7351 nominal with elongated pad for handsoldering. (Body size source: IPC-SM-782 page 72, https://www.pcb-3d.com/wordpress/wp-content/uploads/ipc-sm-782a_amendment_1_and_2.pdf), generated with kicad-footprint-generator")
 		(tags "resistor handsolder")
@@
 	(footprint "Capacitor_SMD:C_0805_2012Metric_Pad1.18x1.45mm_HandSolder"
 		(layer "F.Cu")
-		(at 148.2 108.3)
+		(at 142.7 108.3)
 		(descr "Capacitor SMD 0805 (2012 Metric), square (rectangular) end terminal, IPC_7351 nominal with elongated pad for handsoldering. (Body size source: IPC-SM-782 page 76, https://www.pcb-3d.com/wordpress/wp-content/uploads/ipc-sm-782a_amendment_1_and_2.pdf, https://docs.google.com/spreadsheets/d/1BsfQQcO9C6DZCsRaXUlFlo91Tg2WpOkGARC1WS5S8t0/edit?usp=sharing), generated with kicad-footprint-generator")
 		(tags "capacitor handsolder")
@@
 	(footprint "Button_Switch_SMD:SW_SPDT_CK_JS102011SAQN"
 		(layer "F.Cu")
-		(at 255 98.8 90)
+		(at 205.7 126.6 90)
 		(descr "Sub-miniature slide switch, right-angle, http://www.ckswitches.com/media/1422/js.pdf")
 		(tags "switch spdt")
@@
 		)
 		(pad "1" smd roundrect
-			(at -2.5 -2.75 90)
+			(at -2.5 -2 90)
 			(size 1.25 2.5)
 			(layers "F.Cu" "F.Paste" "F.Mask")
@@
 		)
 		(pad "2" smd roundrect
-			(at 0 -2.75 90)
+			(at 0 -2 90)
 			(size 1.25 2.5)
 			(layers "F.Cu" "F.Paste" "F.Mask")
@@
 		)
 		(pad "3" smd roundrect
-			(at 2.5 -2.75 90)
+			(at 2.5 -2 90)
 			(size 1.25 2.5)
 			(layers "F.Cu" "F.Paste" "F.Mask")
@@
 			(pintype "passive+no_connect")
 		)
+		(pad "NC1" smd roundrect
+			(at -2.5 1 90)
+			(size 1.25 2.5)
+			(layers "F.Cu" "F.Paste" "F.Mask")
+			(roundrect_rratio 0.2)
+			(pinfunction "A")
+			(pintype "passive")
+		)
+		(pad "NC2" smd roundrect
+			(at 0 1 90)
+			(size 1.25 2.5)
+			(layers "F.Cu" "F.Paste" "F.Mask")
+			(roundrect_rratio 0.2)
+			(pinfunction "A")
+			(pintype "passive")
+		)
+		(pad "NC3" smd roundrect
+			(at 2.5 1 90)
+			(size 1.25 2.5)
+			(layers "F.Cu" "F.Paste" "F.Mask")
+			(roundrect_rratio 0.2)
+			(pinfunction "A")
+			(pintype "passive")
+		)
 		(model "${KICAD8_3DMODEL_DIR}/Button_Switch_SMD.3dshapes/SW_SPDT_CK_JS102011SAQN.wrl"
 			(offset
@@
 	(footprint "Resistor_SMD:R_0805_2012Metric_Pad1.20x1.40mm_HandSolder"
 		(layer "F.Cu")
-		(at 148.2 113.3 180)
+		(at 142.7 113.3 180)
 		(descr "Resistor SMD 0805 (2012 Metric), square (rectangular) end terminal, IPC_7351 nominal with elongated pad for handsoldering. (Body size source: IPC-SM-782 page 72, https://www.pcb-3d.com/wordpress/wp-content/uploads/ipc-sm-782a_amendment_1_and_2.pdf), generated with kicad-footprint-generator")
 		(tags "resistor handsolder")
@@
 	(footprint "Jumper:SolderJumper-2_P1.3mm_Open_RoundedPad1.0x1.5mm"
 		(layer "F.Cu")
-		(at 246 99.2 90)
+		(at 202.7 110.7 90)
 		(descr "SMD Solder Jumper, 1x1.5mm, rounded Pads, 0.3mm gap, open")
 		(tags "solder jumper open")
@@
 	(footprint "Capacitor_SMD:C_0805_2012Metric_Pad1.18x1.45mm_HandSolder"
 		(layer "F.Cu")
-		(at 137.2 108.3)
+		(at 148.2 108.3)
 		(descr "Capacitor SMD 0805 (2012 Metric), square (rectangular) end terminal, IPC_7351 nominal with elongated pad for handsoldering. (Body size source: IPC-SM-782 page 76, https://www.pcb-3d.com/wordpress/wp-content/uploads/ipc-sm-782a_amendment_1_and_2.pdf, https://docs.google.com/spreadsheets/d/1BsfQQcO9C6DZCsRaXUlFlo91Tg2WpOkGARC1WS5S8t0/edit?usp=sharing), generated with kicad-footprint-generator")
 		(tags "capacitor handsolder")
@@
 	(footprint "Resistor_SMD:R_0805_2012Metric_Pad1.20x1.40mm_HandSolder"
 		(layer "F.Cu")
-		(at 137.2 113.3 180)
+		(at 148.2 113.3 180)
 		(descr "Resistor SMD 0805 (2012 Metric), square (rectangular) end terminal, IPC_7351 nominal with elongated pad for handsoldering. (Body size source: IPC-SM-782 page 72, https://www.pcb-3d.com/wordpress/wp-content/uploads/ipc-sm-782a_amendment_1_and_2.pdf), generated with kicad-footprint-generator")
 		(tags "resistor handsolder")
@@
 		(width 0.25)
 		(layer "F.Cu")
-		(net 44)
+		(net 45)
 	)
 	(segment
@@
 		(width 0.25)
 		(layer "F.Cu")
-		(net 44)
+		(net 45)
 	)
 	(segment
@@
 	)
 	(group ""
-		(members "2a02f171-f2d2-4439-ac4a-5c8fddf56e64" "76b9ee51-eff9-4cc4-9b0d-877e5395e81d"
-			"96edf072-832a-49fc-854b-2578da9a93e6" "b2c50f23-986b-4f90-b41a-1008f326b574"
-			"c4e692a8-88c2-413e-857f-60074161e125" "cd890b52-7fe5-4a1c-b2b3-76609f4a8f1f"
-			"ed645355-bf49-4681-bc4d-58d7652abd5f" "f1bcb6d6-6e6a-404c-8dca-d95dfc1d7b4d"
-		)
-	)
-	(group ""
