File: PCB/Final_Project_PCB/Final_Project_PCB.kicad_pcb (KiCad board)
At the start: 2 copper layers, 34 parts

Commit message: update again
Connections:
- 01-GND_Breakout1 pad 14: /D-Pad_Down -> /D-Pad_Right
- 01-GND_Breakout1 pad 15: /D-Pad_Left -> /D-Pad_Down
- 01-GND_Breakout1 pad 16: /D-Pad_Right -> /D-Pad_Up
- 01-GND_Breakout1 pad 17: /D-Pad_Up -> /D-Pad_Left
- DevBoardI01-GND1 pad 14: /D-Pad_Down -> /D-Pad_Right
- DevBoardI01-GND1 pad 15: /D-Pad_Left -> /D-Pad_Down
- DevBoardI01-GND1 pad 16: /D-Pad_Right -> /D-Pad_Up
- DevBoardI01-GND1 pad 17: /D-Pad_Up -> /D-Pad_Left
Routing:
- net /D-Pad_Right: track 0.00 -> 23.9 mm
- net /D-Pad_Down: track 0.00 -> 20.9 mm
- net /D-Pad_Up: track 0.00 -> 18.0 mm
- net /D-Pad_Left: track 0.20 -> 15.6 mm
- net /Bottom: track 0.00 -> 12.4 mm
- net /Top: track 0.00 -> 12.2 mm
- net /Select: track 0.00 -> 11.1 mm
Changed lines of the file:
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@@
 			(layers "F.Cu" "F.Paste" "F.Mask")
 			(roundrect_rratio 0.2)
-			(pinfunction "A")
-			(pintype "passive")
 		)
 		(pad "NC2" smd roundrect
@@
 			(layers "F.Cu" "F.Paste" "F.Mask")
 			(roundrect_rratio 0.2)
-			(pinfunction "A")
-			(pintype "passive")
 		)
 		(pad "NC3" smd roundrect
@@
 			(layers "F.Cu" "F.Paste" "F.Mask")
 			(roundrect_rratio 0.2)
-			(pinfunction "A")
-			(pintype "passive")
 		)
 		(model "${KICAD8_3DMODEL_DIR}/Button_Switch_SMD.3dshapes/SW_SPDT_CK_JS102011SAQN.wrl"
@@
 			(layers "*.Cu" "*.Mask")
 			(remove_unused_layers no)
-			(net 47 "/D-Pad_Down")
+			(net 46 "/D-Pad_Right")
 			(pinfunction "Pin_14")
 			(pintype "passive")
@@
 			(layers "*.Cu" "*.Mask")
 			(remove_unused_layers no)
-			(net 45 "/D-Pad_Left")
+			(net 47 "/D-Pad_Down")
 			(pinfunction "Pin_15")
 			(pintype "passive")
@@
 			(layers "*.Cu" "*.Mask")
 			(remove_unused_layers no)
-			(net 46 "/D-Pad_Right")
+			(net 44 "/D-Pad_Up")
 			(pinfunction "Pin_16")
 			(pintype "passive")
@@
 			(layers "*.Cu" "*.Mask")
 			(remove_unused_layers no)
-			(net 44 "/D-Pad_Up")
+			(net 45 "/D-Pad_Left")
 			(pinfunction "Pin_17")
 			(pintype "passive")
@@
 			(layers "*.Cu" "*.Mask")
 			(remove_unused_layers no)
-			(net 47 "/D-Pad_Down")
+			(net 46 "/D-Pad_Right")
 			(pinfunction "Pin_14")
 			(pintype "passive")
@@
 			(layers "*.Cu" "*.Mask")
 			(remove_unused_layers no)
-			(net 45 "/D-Pad_Left")
+			(net 47 "/D-Pad_Down")
 			(pinfunction "Pin_15")
 			(pintype "passive")
@@
 			(layers "*.Cu" "*.Mask")
 			(remove_unused_layers no)
-			(net 46 "/D-Pad_Right")
+			(net 44 "/D-Pad_Up")
 			(pinfunction "Pin_16")
 			(pintype "passive")
@@
 			(layers "*.Cu" "*.Mask")
 			(remove_unused_layers no)
-			(net 44 "/D-Pad_Up")
+			(net 45 "/D-Pad_Left")
 			(pinfunction "Pin_17")
 			(pintype "passive")
@@
 	)
 	(segment
+		(start 158.1625 108.3)
+		(end 158.1625 97.3938)
+		(width 0.5)
+		(layer "F.Cu")
+		(net 9)
+	)
+	(segment
+		(start 158.1625 97.3938)
+		(end 158.3308 97.2255)
+		(width 0.5)
+		(layer "F.Cu")
+		(net 9)
+	)
+	(segment
+		(start 154.5508 106.4117)
+		(end 154.5508 98.4655)
+		(width 0.5)
+		(layer "F.Cu")
+		(net 12)
+	)
+	(segment
+		(start 152.6625 108.3)
+		(end 154.5508 106.4117)
+		(width 0.5)
+		(layer "F.Cu")
+		(net 12)
+	)
+	(segment
+		(start 154.5508 98.4655)
+		(end 155.7908 97.2255)
+		(width 0.5)
+		(layer "F.Cu")
+		(net 12)
+	)
+	(segment
 		(start 132.9308 97.2255)
 		(end 132.9308 92.2255)
@@
 	)
 	(segment
+		(start 163.6625 108.3)
+		(end 163.6625 100.0172)
+		(width 0.5)
+		(layer "F.Cu")
+		(net 19)
+	)
+	(segment
+		(start 163.6625 100.0172)
+		(end 160.8708 97.2255)
+		(width 0.5)
+		(layer "F.Cu")
+		(net 19)
+	)
+	(segment
 		(start 140.5508 97.2255)
 		(end 140.5508 92.2255)
@@
 	)
 	(segment
+		(start 136.1625 108.3)
+		(end 134.9875 107.125)
+		(width 0.5)
+		(layer "F.Cu")
+		(net 44)
+	)
+	(segment
+		(start 134.9875 107.125)
+		(end 132.6703 107.125)
+		(width 0.5)
+		(layer "F.Cu")
+		(net 44)
+	)
+	(segment
+		(start 132.6703 107.125)
+		(end 122.7708 97.2255)
+		(width 0.5)
+		(layer "F.Cu")
+		(net 44)
+	)
+	(segment
 		(start 130.6625 108.3)
 		(end 130.6 108.3)
@@
 	)
 	(segment
+		(start 130.6625 108.3)
+		(end 130.6625 107.6572)
+		(width 0.5)
+		(layer "F.Cu")
+		(net 45)
+	)
+	(segment
+		(start 130.6625 107.6572)
+		(end 120.2308 97.2255)
+		(width 0.5)
+		(layer "F.Cu")
+		(net 45)
+	)
+	(segment
 		(start 130.6 108.3)
 		(end 130.5 108.2)
@@
 	)
 	(segment
+		(start 136.3503 105.725)
+		(end 127.8508 97.2255)
+		(width 0.5)
+		(layer "F.Cu")
+		(net 46)
+	)
+	(segment
+		(start 147.1625 108.3)
+		(end 144.5875 105.725)
+		(width 0.5)
+		(layer "F.Cu")
+		(net 46)
+	)
+	(segment
+		(start 144.5875 105.725)
+		(end 136.3503 105.725)
+		(width 0.5)
+		(layer "F.Cu")
+		(net 46)
+	)
+	(segment
+		(start 141.6625 108.3)
+		(end 139.7875 106.425)
+		(width 0.5)
+		(layer "F.Cu")
+		(net 47)
+	)
+	(segment
+		(start 134.5103 106.425)
+		(end 125.3108 97.2255)
+		(width 0.5)
+		(layer "F.Cu")
+		(net 47)
+	)
+	(segment
+		(start 139.7875 106.425)
+		(end 134.5103 106.425)
+		(width 0.5)
+		(layer "F.Cu")
+		(net 47)
+	)
+	(segment

Commit message: LDC PCB
Routing:
- net /Vin(3.3): track 0.00 -> 118.3 mm
- net Net-(Amplifier1-Pin_4): track 0.00 -> 78.8 mm
- net /Bottom_Button: track 0.00 -> 38.2 mm
- net /Select_Button: track 0.04 -> 34.2 mm
- net /Down: track 0.00 -> 31.2 mm
- net /Right: track 0.00 -> 20.6 mm
- net /Left: track 0.00 -> 19.7 mm
- net /Top_Button: track 0.00 -> 14.5 mm
- net /Up: track 0.00 -> 10.6 mm
- net GND: track 0.00 -> 8.37 mm
- net (no net): track 0.00 -> 1.65 mm
