File: PCB/Final_Project_PCB/Final_Project_PCB.kicad_pcb (KiCad board)
At the start: 2 copper layers, 34 parts

Commit message: updates againnnn
Parts:
- added LCD1: Conn_01x14_Pin, Connector_PinHeader_2.54mm:PinHeader_1x14_P2.54mm_Vertical, F.Cu at (216.3, 63.7)

Commit message: Save before filling in front and back planes with copper
Parts:
- removed OnOff1: SW_SPDT, Button_Switch_SMD:SW_SPDT_CK_JS102011SAQN
- added MNT1: MountingHole_5.3mm_M5_ISO7380_Pad_TopBottom, MountingHole:MountingHole_5.3mm_M5_ISO7380_Pad_TopBottom, F.Cu at (172.7, 89.7)
- added MNT2: MountingHole_5.3mm_M5_ISO7380_Pad_TopBottom, MountingHole:MountingHole_5.3mm_M5_ISO7380_Pad_TopBottom, F.Cu at (198.0, 151.0)
- added MNT3: MountingHole_5.3mm_M5_ISO7380_Pad_TopBottom, MountingHole:MountingHole_5.3mm_M5_ISO7380_Pad_TopBottom, F.Cu at (120.0, 151.0)
- added SS1: SW_Slide_DPDT, Button_Switch_SMD:SW_DPDT_CK_JS202011JCQN, F.Cu at (205.5, 126.5)
- moved LCD1 32.3 mm to (206.0, 94.3), turned to 180 degrees
- moved Top_button1 0.20 mm to (178.3, 123.6)
- moved Bottom_button1 0.11 mm to (178.6, 143.7)
- moved Select1 0.10 mm to (188.6, 133.6)
Connections:
- 46-GND_Breakout1 pad 3: /RX0 -> /IO44
- 46-GND_Breakout1 pad 4: /TX0 -> /IO43
- DevBoardIO46-GND1 pad 3: /RX0 -> /IO44
- DevBoardIO46-GND1 pad 4: /TX0 -> /IO43
Routing:
- net /+: track 0.00 -> 172.4 mm, vias 0 -> 1
- net /IO33: track 5.00 -> 117.5 mm
- net /IO47: track 5.00 -> 112.9 mm
- net /IO35: track 5.00 -> 102.2 mm
- net /IO37: track 5.00 -> 96.5 mm
- net /IO36: track 5.00 -> 96.0 mm
- net /IO34: track 5.00 -> 94.5 mm, vias 0 -> 3
- net /Vin(3.3): track 118.3 -> 200.5 mm
- net /IO41: track 5.00 -> 81.9 mm
- net /IO43: track 0.00 -> 73.0 mm
- net /IO42: track 5.00 -> 77.5 mm
- net Net-(JSTBattery1-Pin_2): track 0.00 -> 71.3 mm, vias 0 -> 2
- net /IO44: track 0.00 -> 68.5 mm
- net /IO45: track 5.00 -> 64.0 mm
- net /IO46: track 5.00 -> 59.0 mm
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Other:
- board outline added: 98 x 111 mm

Commit message: Final PCB Update - Pending Review
Parts:
- renumbered GenConnector1 to BatToBoard1
Connections:
- LCD1 pad 1: /Vin(3.3) -> /+
Routing:
- net /+: track 172.4 -> 185.3 mm, vias 1 -> 2
- net /Vin(3.3): track 200.5 -> 205.3 mm
- net GND: vias 0 -> 9
- added copper zone on B.Cu, net GND
- added copper zone on F.Cu, net GND
Other:
- board text added: "UCSD ECE 196 - Engineering Hands-On Group Project Melissa De La Cruz, Giselle Mendoza, Dustin Miller"
- board text removed: "No debounce for power switch, switch to J1 and amp okay[p;k,"
- board text removed: "Poth planes are ground planes"
- board text removed: "put RC circuits as close to the microcontroller as possible"
